Commit message: Launch file and started gazebo

File: description/robot_core.xacro (robot description, xacro)
@@ -45,4 +45,7 @@
         </xacro:inertial_box>
     </link>
+    <gazebo reference="chassis">
+            <material>Gazebo/Blue</material>
+    </gazebo>
     <!-- BRAIN BOX -->
     <joint name="brainbox_joint" type="fixed">
@@ -70,4 +73,7 @@
         </xacro:inertial_box>
     </link>
+    <gazebo reference="brainbox">
+            <material>Gazebo/Green</material>
+    </gazebo>
     <!-- BUMPER -->
     <joint name="bumper_joint" type="fixed">
@@ -92,4 +98,7 @@
         </xacro:inertial_cylinder>
     </link>
+    <gazebo reference="bumper">
+            <material>Gazebo/White</material>
+    </gazebo>
     <!-- BACK -->
     <!-- BACK LEFT WHEEL LINK -->
@@ -116,4 +125,7 @@
         </xacro:inertial_cylinder>
     </link>
+    <gazebo reference="back_left_wheel">
+            <material>Gazebo/Black</material>
+    </gazebo>
         <!-- BACK RIGHT WHEEL LINK -->
     <joint name="back_right_wheel_joint" type="continuous">
@@ -139,4 +151,7 @@
         </xacro:inertial_cylinder>
     </link>
+    <gazebo reference="back_right_wheel">
+            <material>Gazebo/Black</material>
+    </gazebo>
         <!-- FRONT -->
         <!-- FRONT LEFT WHEEL LINK -->
@@ -163,4 +178,7 @@
         </xacro:inertial_cylinder>
     </link>
+    <gazebo reference="front_left_wheel">
+            <material>Gazebo/Black</material>
+    </gazebo>
         <!-- FRONT RIGHT WHEEL LINK -->
     <joint name="front_right_wheel_joint" type="continuous">
@@ -186,3 +204,6 @@
         </xacro:inertial_cylinder>
     </link>
+    <gazebo reference="front_right_wheel">
+            <material>Gazebo/Black</material>
+    </gazebo>
 </robot>
